Commit message: Updated the Gazebo world and cart code

File: autocart_ws/install/autocart_sim/share/autocart_sim/models/cart.urdf (robot description, URDF)
Before this commit: robot autocart, 3 links, 2 joints
Links:
- removed link camera_link
- removed link imu_link
- added link basket; visual box size=0.55 0.38 0.35
- added link handle_bar; visual cylinder length=0.38 radius=0.025
- added link wheel_fl; visual cylinder length=0.05 radius=0.07
- added link wheel_fr; visual cylinder length=0.05 radius=0.07
- added link wheel_rl; visual cylinder length=0.05 radius=0.07
- added link wheel_rr; visual cylinder length=0.05 radius=0.07
- link base_link: mass 15.0 -> 18.0; geometry collision box size=0.7 0.45 0.16; visual box size=0.7 0.45 0.16
Joints:
- removed joint camera_joint
- removed joint imu_joint
- added joint basket_joint: type fixed, parent base_link, child basket
- added joint handle_joint: type fixed, parent base_link, child handle_bar
- added joint joint_wheel_fl: type fixed, parent base_link, child wheel_fl
- added joint joint_wheel_fr: type fixed, parent base_link, child wheel_fr
- added joint joint_wheel_rl: type fixed, parent base_link, child wheel_rl
- added joint joint_wheel_rr: type fixed, parent base_link, child wheel_rr
