Commit message: Add Gazebo Harmonic support with differential drive and ROS2 Jazzy bridge

File: autocart_ws/src/autocart_sim/autocart_sim/models/cart.urdf (robot description, URDF)
Before this commit: robot autocart, 3 links, 2 joints
Links:
- added link front_caster, mass 0.5; collision sphere radius=0.05; visual sphere radius=0.05
- added link left_wheel, mass 1.0; collision cylinder length=0.05 radius=0.1; visual cylinder length=0.05 radius=0.1
- added link right_wheel, mass 1.0; collision cylinder length=0.05 radius=0.1; visual cylinder length=0.05 radius=0.1
Joints:
- added joint front_caster_joint: type fixed, parent base_link, child front_caster, origin xyz=0.3 0 0.05 rpy=0 0 0
- added joint left_wheel_joint: type continuous, parent base_link, child left_wheel, origin xyz=-0.2 0.35 0.1 rpy=0 0 0, axis 0 1 0
- added joint right_wheel_joint: type continuous, parent base_link, child right_wheel, origin xyz=-0.2 -0.35 0.1 rpy=0 0 0, axis 0 1 0
